File: EAGLE/PCB Class.brd (EAGLE design)
At the start: 100 x 80 mm, 0 parts

Commit message: Updates to schematics
Parts:
- added BUTTON0, BUTTON1, BUTTON2, BUTTON3, BUTTON4, BUTTON5: (no value), ENGI301_PCB_design_project:BUTTON
- added BUZZER: (no value), ENGI301_PCB_design_project:SEM-1203(42)
- added C1, C2, C3: (no value), ENGI301_PCB_design_project:C0402
- added LED0, LED1, LED2: (no value), ENGI301_PCB_design_project:LTST-C191TBKT
- added MOD, MOD1: MOD-LED8X8RGB-CONN, ENGI301_PCB_design_project:FE06W
- added MPU: (no value), ENGI301_PCB_design_project:QFN-3MMX3MM
- added POCKETBEAGLE: POCKETBEAGLE, ENGI301_PCB_design_project:POCKETBEAGLE
- added R1, R2, R3: 1K, ENGI301_PCB_design_project:R0603
- added R10, R11, R4, R5, R6, R7, R8, R9: 3K, ENGI301_PCB_design_project:R0603
Connections:
- new net 8X8CLK: MOD.2, POCKETBEAGLE.8
- new net 8X8MISO: MOD.4, MOD1.4, POCKETBEAGLE.63
- new net 8X8MOSI: MOD.3, MOD1.3, POCKETBEAGLE.61
- new net BUTTON0: POCKETBEAGLE.48, R6.2
- new net BUTTON1: POCKETBEAGLE.20, R7.2
- new net BUTTON2: POCKETBEAGLE.55, R8.2
- new net BUTTON3: BUTTON3.P$1, POCKETBEAGLE.58, R9.2
- new net BUTTON4: BUTTON4.P$1, POCKETBEAGLE.54, R10.2
- new net BUTTON5: POCKETBEAGLE.60, R11.2
- new net GND: BUZZER.P$2, C1.2, C2.2, C3.2, MPU.18, MPU.20
- new net N$1: MPU.10
- new net N$11: LED2.P$1, R3.1
- new net N$12: R1.1
- new net N$13: LED1.P$1, R2.1
- new net N$15: BUZZER.P$1, POCKETBEAGLE.37
- new net N$16: BUTTON0.P$2
- new net N$17: R4.2
- new net N$18: R5.2
- new net N$19: BUTTON1.P$2
- new net N$2: MPU.24, R5.1
- new net N$20: BUTTON5.P$2
- new net N$22: BUTTON3.P$2
- new net N$23: BUTTON2.P$2
- new net N$24: MOD.5, MOD.6, MOD1.6
- new net N$25: POCKETBEAGLE.24
- new net N$3: MPU.23, R4.1
- new net N$5: R2.2
- new net N$6: POCKETBEAGLE.44, R3.2
- new net N$7: MPU.1, MPU.22
- new net N$8: LED0.P$2
- new net SYS_VDD1_3P3V: C1.1, C2.1, MOD.1, MOD1.1, MPU.13, MPU.8, POCKETBEAGLE.14, POCKETBEAGLE.49, POCKETBEAGLE.59, R6.1, R7.1
Other:
- board size 100 x 80 mm -> 152.4 x 152.4 mm
