File: EAGLE/PCB Class.brd (EAGLE design)
At the start: 152.4 x 63.5 mm, 32 parts

Commit message: FINAL PROJECT 2A MEZMUR
Parts:
- C1: value (none) -> 10nF
- C2, C3: value (none) -> 0.1uF
- moved R5 24.1 mm to (44.5, 49.5)
- moved MPU 23.4 mm to (49.5, 44.5)
- moved R10 22.9 mm to (2.54, 39.4)
- moved C1 16.3 mm to (59.7, 44.5), turned to 90 degrees
- moved R4 16.1 mm to (53.3, 49.5)
- moved R8 15.5 mm to (35.6, 26.7), turned to 90 degrees
- moved C3 13.7 mm to (62.2, 38.1), turned to 270 degrees
- moved R9 10.5 mm to (16.5, 11.4)
- moved C2 8.03 mm to (71.1, 41.9), turned to 90 degrees
- moved R11 7.62 mm to (19.1, 34.3), turned to 90 degrees
- moved BUTTON1 2.54 mm to (24.5, 46.4)
- moved BUZZER 2.54 mm to (80.0, 47.0), turned to 180 degrees
- moved R6 2.54 mm to (40.6, 39.4)
Connections:
- net 8X8CLK1: now also MOD1.2
- net GND: now also MOD1.5
- net N$1: now also C3.1
Routing:
- net SYS_VDD1_3P3V: track 0.00 -> 178.7 mm
- net BUTTON4: track 0.00 -> 154.2 mm
- net BUTTON3: track 0.00 -> 137.8 mm
- net BUTTON5: track 0.00 -> 137.7 mm
- net 8X8CLK1: track 0.00 -> 123.3 mm
- net GND: track 0.00 -> 121.6 mm, vias 0 -> 1
- net BUTTON1: track 0.00 -> 121.4 mm
- net 8X8CS1: track 0.00 -> 119.3 mm
- net BUTTON0: track 0.00 -> 118.5 mm
- net 8X8MOSI1: track 0.00 -> 111.9 mm
- net BUTTON2: track 0.00 -> 96.5 mm
- net 8X8CS: track 0.00 -> 56.2 mm
- net 8X8MOSI: track 0.00 -> 51.7 mm
- net 8X8CLK: track 0.00 -> 51.7 mm
- net N$15: track 0.00 -> 24.5 mm
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- added copper zone on layer 2, net GND
- added copper zone on layer 15, net VDD_3P3V
- removed copper zone on layer 2, net N$4
- removed copper zone on layer 15, net N$9
Other:
- board text added: "CM"
- board text added: "Christina Mezmur ENGI 301 PCB"
