File: EAGLE/PCB Class.sch (EAGLE design)
At the start: 0 parts

Commit message: Updates to schematics
Parts:
- added BUTTON0, BUTTON1, BUTTON2, BUTTON3, BUTTON4, BUTTON5: (no value), ENGI301_PCB_design_project:BUTTON
- added BUZZER: (no value), ENGI301_PCB_design_project:SEM-1203(42)
- added C1, C2, C3: (no value), ENGI301_PCB_design_project:C_C0402
- added LED0, LED1, LED2: (no value), ENGI301_PCB_design_project:LTST-C191TBKT
- added MOD, MOD1: MOD-LED8X8RGB-CONN, ENGI301_PCB_design_project:MOD-LED8X8RGB-CONN
- added MPU: (no value), ENGI301_PCB_design_project:MPU-9250
- added POCKETBEAGLE: POCKETBEAGLE, ENGI301_PCB_design_project:POCKETBEAGLE
- added R1, R2, R3: 1K, ENGI301_PCB_design_project:R_R0603
- added R10, R11, R4, R5, R6, R7, R8, R9: 3K, ENGI301_PCB_design_project:R_R0603
Connections:
- new net 8X8CLK: MOD.DATA_SCK_IN, POCKETBEAGLE.SPI0.CLK
- new net 8X8MISO: MOD.DATA_LINE_IN, MOD1.DATA_LINE_IN, POCKETBEAGLE.SPI0.MISO
- new net 8X8MOSI: MOD.DATA_LATCH_IN/#MCLR, MOD1.DATA_LATCH_IN/#MCLR, POCKETBEAGLE.SPI0.MOSI
- new net BUTTON0: POCKETBEAGLE.PWR.BTN, R6.2
- new net BUTTON1: POCKETBEAGLE.GPIO20, R7.2
- new net BUTTON2: POCKETBEAGLE.GPIO27, R8.2
- new net BUTTON3: BUTTON3.P$1, POCKETBEAGLE.GPIO46, R9.2
- new net BUTTON4: BUTTON4.P$1, POCKETBEAGLE.GPIO47, R10.2
- new net BUTTON5: POCKETBEAGLE.GPIO48, R11.2
- new net GND: BUZZER.-, C1.2, C2.2, C3.2, MPU.GND, MPU.RESV@2
- new net N$1: MPU.REGOUT
- new net N$11: LED2.P$1, R3.1
- new net N$12: R1.1
- new net N$13: LED1.P$1, R2.1
- new net N$15: BUZZER.+, POCKETBEAGLE.PWM1A
- new net N$16: BUTTON0.P$2
- new net N$17: R4.2
- new net N$18: R5.2
- new net N$19: BUTTON1.P$2
- new net N$2: MPU.SDA/SDI, R5.1
- new net N$20: BUTTON5.P$2
- new net N$22: BUTTON3.P$2
- new net N$23: BUTTON2.P$2
- new net N$24: MOD.GND@1, MOD.GND@2, MOD1.GND@2
- new net N$25: POCKETBEAGLE.VOUT@1
- new net N$3: MPU.SCL/SCLK, R4.1
- new net N$5: R2.2
- new net N$6: POCKETBEAGLE.GPIO60, R3.2
- new net N$7: MPU.NCS, MPU.RESV@0
- new net N$8: LED0.P$2
- new net SYS_VDD1_3P3V: C1.1, C2.1, MOD.5V, MOD1.5V, MPU.VDD, MPU.VDD10, POCKETBEAGLE.3.3V@1, POCKETBEAGLE.3.3V@2, POCKETBEAGLE.VOUT@2, R6.1, R7.1
Other:
- note added: "8 X 8 LED ARRAY"
- note added: "9-AXIS IMU"
- note added: "BUTTONS"
- note added: "BUZZER"
- note added: "Christina Mezmur"
- note added: "LED ARRAYS"
- note added: "LEDs"
- note added: "POCKET BEAGLE"
